File: Hardware/MidiSwitchPCB/MidiSwitchPCB.brd (EAGLE design)
At the start: 160 x 100 mm, 65 parts, among them IC1 74AHC1G04DBV, IC2 74AHC1G04DBV, K1 APF30212C, K2 APF30212C, K3 APF30212C, K4 APF30212C, K5 APF30212C, K6 APF30212C, K7 APF30212C, K8 APF30212C, Q1 BSS123, Q2 BSS123, Q3 BSS123, Q4 BSS123, Q5 BSS123, Q6 BSS123, Q7 BSS123, Q8 BSS123, X1 1503_09, X2 1503_09, X3 1503_09, X4 1503_09

Commit message: added some links to partlist
Parts:
- removed IC1, IC2: 74AHC1G04DBV, 74xx-little-de:SOT23-5
- added IC3: 74LVC2G04GW,125, 74LVC2G04GW_125:SOT65P210X110-6N
- added R18, R19: 0R, rcl:R0603
Connections:
- new net N$58: PS1.8, R18.2, R19.1
- new net VCC_3_3: IC3.5, OK1.8, R3.2, R5.2
- new net VCC_6-8: C1.1, C2.+, C3.1, C4.1, CN6.8, D2.C, D3.C, D4.C, D5.C, D6.C, D7.C, D8.C, D9.C, K1.1, K2.1, K3.1, K4.1, K5.1, K6.1, K7.1, K8.1, PS1.16, PS1.17, R14.1, R15.2
- net GND: now also IC3.2, R19.2; no longer IC1.3, IC2.3
- net MIDI_RX: now also IC3.3; no longer IC1.2
- net N$1: now also IC3.1, IC3.4; no longer IC1.4, IC2.2
- net N$11: now also IC3.6; no longer IC2.4
- net N$53: now also R18.1
- net VCC: now also CN6.4; no longer C1.1, C2.+, C3.1, C4.1, CN6.8, D2.C, D3.C, D4.C, D5.C, D6.C, D7.C, D8.C, D9.C, IC1.5, IC2.5, K1.1, K2.1, K3.1, K4.1, K5.1, K6.1, K7.1, K8.1, OK1.8, PS1.16, PS1.17, R14.1, R15.2, R3.2, R5.2
