File: Hardware/MidiSwitchPCB/MidiSwitchPCB.sch (EAGLE design)
At the start: 65 parts, among them IC1 74AHC1G04DBV, IC2 74AHC1G04DBV, K1 APF30212C, K2 APF30212C, K3 APF30212C, K4 APF30212C, K5 APF30212C, K6 APF30212C, K7 APF30212C, K8 APF30212C, Q1 BSS123, Q2 BSS123, Q3 BSS123, Q4 BSS123, Q5 BSS123, Q6 BSS123, Q7 BSS123, Q8 BSS123, X1 1503_09, X2 1503_09, X3 1503_09, X4 1503_09

Commit message: added some links to partlist
Parts:
- removed IC1, IC2: 74AHC1G04DBV, 74xx-little-de:74AHC1G04DBV
- added IC3: 74LVC2G04GW,125, 74LVC2G04GW_125:74LVC2G04GW,125
- added R18, R19: 0R, rcl:R-EU_R0603
Connections:
- new net N$58: PS1.IGN_PWRL, R18.2, R19.1
- new net VCC_3_3: IC3.VCC, OK1.VCC, R3.2, R5.2
- new net VCC_6-8: C1.1, C2.+, C3.1, C4.1, CN6.8, D2.C, D3.C, D4.C, D5.C, D6.C, D7.C, D8.C, D9.C, K11.1, K21.1, K31.1, K41.1, K51.1, K61.1, K71.1, K81.1, PS1.VOUT, PS1.VOUT_SENSE, R14.1, R15.2
- net GND: now also IC3.GND, R19.2
- net MIDI_RX: now also IC3.2A; no longer IC1A.I
- net N$1: now also IC3.1A, IC3.2Y; no longer IC1A.O, IC2A.I
- net N$11: now also IC3.1Y; no longer IC2A.O
- net N$53: now also R18.1
- net VCC: now also CN6.4; no longer C1.1, C2.+, C3.1, C4.1, CN6.8, D2.C, D3.C, D4.C, D5.C, D6.C, D7.C, D8.C, D9.C, K11.1, K21.1, K31.1, K41.1, K51.1, K61.1, K71.1, K81.1, OK1.VCC, PS1.VOUT, PS1.VOUT_SENSE, R14.1, R15.2, R3.2, R5.2
Other:
- note removed: "Pull up mit zener diode"
- moved on the sheet: C7
