File: Hardware/MidiSwitchPCB/MidiSwitchPCB.sch (EAGLE design)
At the start: 78 parts, among them IC3 74LVC2G04GW,125, J1 694108106102, J2 NMJ6HCD2, J3 NMJ6HCD2, J4 NMJ6HCD2, J5 NMJ6HCD2, Q1 BSS123, Q2 BSS123, Q3 BSS123, Q4 BSS123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

Commit message: finished layout reworking
Parts:
- IC3: value 74LVC2G04GW,125 -> 74LVC2G04GW
- PS1: value TPS55160QPWPTQ1 -> TPS55160
- U$10, U$3, U$4, U$5, U$6, U$7, U$8, U$9: value G6L-1F-TR_DC5-NEW -> Relay
Connections:
- net GND: now also CN5.7, CN6.6, CN6.7
Changed lines of the file:
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@@
 <setting verticaltext="up"/>
 </settings>
-<grid distance="0.01" unitdist="mm" unit="mm" style="lines" multiple="10" display="yes" altdistance="0.01" altunitdist="mm" altunit="mm"/>
+<grid distance="0.01" unitdist="mm" unit="mm" style="lines" multiple="10" display="no" altdistance="0.01" altunitdist="mm" altunit="mm"/>
 <layers>
 <layer number="1" name="Top" color="4" fill="1" visible="no" active="no"/>
@@
 </variantdefs>
 <classes>
-<class number="0" name="default" width="0.4064" drill="1.016">
+<class number="0" name="default" width="0.1524" drill="0.3556">
 <clearance class="0" value="0.1524"/>
 </class>
-<class number="1" name="Power" width="1.016" drill="1.016">
+<class number="1" name="Power" width="1.016" drill="0.3556">
 <clearance class="1" value="0.4064"/>
 </class>
-<class number="2" name="Signal" width="0.1524" drill="0.6096">
+<class number="2" name="Signal" width="0.1524" drill="0.3556">
 <clearance class="2" value="0.1524"/>
 </class>
-<class number="3" name="WideIsolation" width="0.4064" drill="1.016">
+<class number="3" name="WideIsolation" width="0.1524" drill="0.3556">
 <clearance class="3" value="2.032"/>
 </class>
-<class number="4" name="ESD_Critical" width="0.4064" drill="1.016">
+<class number="4" name="ESD_Critical" width="0.1524" drill="0.3556">
 <clearance class="4" value="0.6096"/>
 </class>
@@
 <part name="SUPPLY11" library="supply2" deviceset="GND" device=""/>
 <part name="C2" library="rcl" deviceset="CPOL-EU" device="153CLV-1012"/>
-<part name="PS1" library="TPS55160QPWPTQ1" deviceset="TPS55160QPWPTQ1" device=""/>
+<part name="PS1" library="TPS55160QPWPTQ1" deviceset="TPS55160QPWPTQ1" device="" value="TPS55160"/>
 <part name="R_PG" library="rcl" deviceset="R-EU_" device="R0603" value="10-100k"/>
 <part name="R15" library="rcl" deviceset="R-EU_" device="R0603" value="800k"/>
@@
 <part name="SUPPLY19" library="supply2" deviceset="GND" device=""/>
 <part name="C_REG" library="rcl" deviceset="C-EU" device="C0805" value="4.7 µF"/>
-<part name="IC3" library="74LVC2G04GW_125" deviceset="74LVC2G04GW,125" device=""/>
+<part name="IC3" library="74LVC2G04GW_125" deviceset="74LVC2G04GW,125" device="" value="74LVC2G04GW"/>
 <part name="VCC_3_3" library="supply1" deviceset="VCC" device="" value="VCC_3_3"/>
 <part name="SUPPLY20" library="supply2" deviceset="GND" device=""/>
@@
 <part name="R27" library="rcl" deviceset="R-EU_" device="R0603" value="61"/>
 <part name="J1" library="SamacSys_Parts" deviceset="694108106102" device=""/>
-<part name="U$3" library="SamacSys_Parts" deviceset="G6L-1F-TR_DC5-NEW" device=""/>
-<part name="U$4" library="SamacSys_Parts" deviceset="G6L-1F-TR_DC5-NEW" device=""/>
-<part name="U$5" library="SamacSys_Parts" deviceset="G6L-1F-TR_DC5-NEW" device=""/>
-<part name="U$6" library="SamacSys_Parts" deviceset="G6L-1F-TR_DC5-NEW" device=""/>
-<part name="U$7" library="SamacSys_Parts" deviceset="G6L-1F-TR_DC5-NEW" device=""/>
-<part name="U$8" library="SamacSys_Parts" deviceset="G6L-1F-TR_DC5-NEW" device=""/>
-<part name="U$9" library="SamacSys_Parts" deviceset="G6L-1F-TR_DC5-NEW" device=""/>
-<part name="U$10" library="SamacSys_Parts" deviceset="G6L-1F-TR_DC5-NEW" device=""/>
+<part name="U$3" library="SamacSys_Parts" deviceset="G6L-1F-TR_DC5-NEW" device="" value="Relay"/>
+<part name="U$4" library="SamacSys_Parts" deviceset="G6L-1F-TR_DC5-NEW" device="" value="Relay"/>
+<part name="U$5" library="SamacSys_Parts" deviceset="G6L-1F-TR_DC5-NEW" device="" value="Relay"/>
+<part name="U$6" library="SamacSys_Parts" deviceset="G6L-1F-TR_DC5-NEW" device="" value="Relay"/>
+<part name="U$7" library="SamacSys_Parts" deviceset="G6L-1F-TR_DC5-NEW" device="" value="Relay"/>
+<part name="U$8" library="SamacSys_Parts" deviceset="G6L-1F-TR_DC5-NEW" device="" value="Relay"/>
+<part name="U$9" library="SamacSys_Parts" deviceset="G6L-1F-TR_DC5-NEW" device="" value="Relay"/>
+<part name="U$10" library="SamacSys_Parts" deviceset="G6L-1F-TR_DC5-NEW" device="" value="Relay"/>
 <part name="F1" library="rcl" deviceset="R-EU_" device="R0603" value="1A"/>
 <part name="D10" library="diode" deviceset="BAS70-06" device=""/>
@@
 <part name="SUPPLY28" library="supply2" deviceset="GND" device=""/>
 <part name="B1" library="rectifier" deviceset="MB*S" device="" technology="1"/>
+<part name="SUPPLY29" library="supply2" deviceset="GND" device=""/>
+<part name="SUPPLY30" library="supply2" deviceset="GND" device=""/>
 </parts>
 <sheets>
@@
 <instance part="SUPPLY28" gate="GND" x="218.94" y="-79.46"/>
 <instance part="B1" gate="G$1" x="310.01" y="12.16" rot="MR90"/>
+<instance part="SUPPLY29" gate="GND" x="148.87" y="82.46"/>
+<instance part="SUPPLY30" gate="GND" x="346.47" y="73.35"/>
 </instances>
 <busses>
@@
 </segment>
 </net>
-<net name="GND" class="0">
+<net name="GND" class="1">
 <segment>
 <wire x1="72.64" y1="78.46" x2="72.64" y2="75.21" width="0.1524" layer="91"/>
@@
 <junction x="190.05" y="-75.61"/>
 </segment>
+<segment>
+<pinref part="CN5" gate="A" pin="7"/>
+<pinref part="SUPPLY29" gate="GND" pin="GND"/>
+<wire x1="148.87" y1="92.19" x2="148.87" y2="85" width="0.1524" layer="91"/>
+</segment>
+<segment>
+<pinref part="SUPPLY30" gate="GND" pin="GND"/>
+<wire x1="346.47" y1="75.89" x2="346.47" y2="82.41" width="0.1524" layer="91"/>
+<pinref part="CN6" gate="A" pin="7"/>
+<wire x1="346.47" y1="82.41" x2="346.48" y2="82.41" width="0.1524" layer="91"/>
+<pinref part="CN6" gate="A" pin="6"/>
+<wire x1="346.48" y1="82.41" x2="353.31" y2="82.41" width="0.1524" layer="91"/>
+<wire x1="353.31" y1="84.95" x2="346.47" y2="84.95" width="0.1524" layer="91"/>
+<wire x1="346.47" y1="84.95" x2="346.47" y2="82.41" width="0.1524" layer="91"/>
+<junction x="346.48" y="82.41"/>
+</segment>
 </net>
 <net name="N$5" class="0">
@@
 </segment>
 </net>
-<net name="N$56" class="0">
+<net name="N$56" class="1">
 <segment>
 <pinref part="C_BST1" gate="G$1" pin="2"/>

Commit message: Debugged pin configuration causing device to be stuck in initialization. Debug code needs to be removed. Reverted pin config to previous pin config. Bug needs to be fixed in HW
Parts:
- renumbered U$1 to MIDI-IN, U$2 to MIDI-THRU
Changed lines of the file:
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@@
 <setting verticaltext="up"/>
 </settings>
-<grid distance="0.01" unitdist="mm" unit="mm" style="lines" multiple="10" display="no" altdistance="0.01" altunitdist="mm" altunit="mm"/>
+<grid distance="0.1" unitdist="inch" unit="inch" style="lines" multiple="1" display="no" altdistance="0.01" altunitdist="inch" altunit="inch"/>
 <layers>
 <layer number="1" name="Top" color="4" fill="1" visible="no" active="no"/>
@@
 </classes>
 <parts>
-<part name="U$2" library="MidiSwitchParts" deviceset="MIDI_CONNECTOR" device=""/>
-<part name="U$1" library="MidiSwitchParts" deviceset="MIDI_CONNECTOR" device=""/>
+<part name="MIDI-THRU" library="MidiSwitchParts" deviceset="MIDI_CONNECTOR" device=""/>
+<part name="MIDI-IN" library="MidiSwitchParts" deviceset="MIDI_CONNECTOR" device=""/>
 <part name="OK1" library="6N138S" deviceset="6N138S" device=""/>
 <part name="D1" library="diode" deviceset="BAS70" device=""/>
@@
 </plain>
 <instances>
-<instance part="U$2" gate="G$1" x="13.14" y="53.42"/>
-<instance part="U$1" gate="G$1" x="12.5" y="82.6"/>
+<instance part="MIDI-THRU" gate="G$1" x="13.14" y="53.42"/>
+<instance part="MIDI-IN" gate="G$1" x="12.5" y="82.6"/>
 <instance part="OK1" gate="G$1" x="57.82" y="83.54"/>
 <instance part="D1" gate="1" x="43.32" y="82.01" rot="R90"/>
@@
 <net name="N$3" class="3">
 <segment>
-<pinref part="U$1" gate="G$1" pin="P$4"/>
+<pinref part="MIDI-IN" gate="G$1" pin="P$4"/>
 <wire x1="25.5" y1="85.6" x2="28.2" y2="85.6" width="0.1524" layer="91"/>
 <wire x1="28.2" y1="85.6" x2="31.2" y2="88.6" width="0.1524" layer="91"/>
@@
 <wire x1="45.12" y1="78.46" x2="43.33" y2="78.44" width="0.1524" layer="91"/>
 <wire x1="43.33" y1="78.44" x2="43.32" y2="79.47" width="0.1524" layer="91"/>
-<pinref part="U$1" gate="G$1" pin="P$5"/>
+<pinref part="MIDI-IN" gate="G$1" pin="P$5"/>
 <wire x1="25.5" y1="79.6" x2="31.52" y2="79.6" width="0.1524" layer="91"/>
 <wire x1="31.52" y1="79.6" x2="31.55" y2="79.56" width="0.1524" layer="91"/>
@@
 <segment>
 <wire x1="25.5" y1="91.6" x2="29.5" y2="91.6" width="0.1524" layer="91"/>
-<pinref part="U$1" gate="G$1" pin="P$7"/>
+<pinref part="MIDI-IN" gate="G$1" pin="P$7"/>
 <wire x1="29.5" y1="91.6" x2="29.5" y2="73.61" width="0.1524" layer="91"/>
 <wire x1="29.5" y1="73.61" x2="29.5" y2="73.6" width="0.1524" layer="91"/>
 <wire x1="25.5" y1="73.6" x2="29.5" y2="73.6" width="0.1524" layer="91"/>
-<pinref part="U$1" gate="G$1" pin="P$6"/>
+<pinref part="MIDI-IN" gate="G$1" pin="P$6"/>
 <pinref part="SUPPLY2" gate="GND" pin="GND"/>
 <junction x="29.5" y="73.61"/>
@@
 <net name="N$5" class="0">
 <segment>
-<pinref part="U$2" gate="G$1" pin="P$4"/>
+<pinref part="MIDI-THRU" gate="G$1" pin="P$4"/>
 <pinref part="R5" gate="G$1" pin="1"/>
 <wire x1="26.14" y1="56.42" x2="28.42" y2="56.42" width="0.1524" layer="91"/>
@@
 <pinref part="R4" gate="G$1" pin="2"/>
 <wire x1="26.14" y1="50.42" x2="28.28" y2="50.42" width="0.1524" layer="91"/>
-<pinref part="U$2" gate="G$1" pin="P$5"/>
-</segment>
-</net>
+<pinref part="MIDI-THRU" gate="G$1" pin="P$5"/>
+</segment>
+</net>
